Commit message: fixed xacro file view, added directions 2 run robot view in rviz2

File: src/base/robot urdf models/f1tent.urdf (robot description, URDF)
Before this commit: robot racecar, 8 links, 7 joints
Links:
- link ego_racecar/back_left_wheel: geometry visual cylinder length=0.02 radius=0.05
- link ego_racecar/back_right_wheel: geometry visual cylinder length=0.02 radius=0.05
- link ego_racecar/base_link: geometry visual box size=0.25 0.2 0.2
- link ego_racecar/front_left_wheel: geometry visual cylinder length=0.02 radius=0.05
- link ego_racecar/front_right_wheel: geometry visual cylinder length=0.02 radius=0.05
Joints:
- removed joint $base_to_back_left_wheel
- added joint base_to_back_left_wheel: type continuous, parent ego_racecar/base_link, child ego_racecar/back_left_wheel, origin xyz=0 0.11 0.05, axis 0 1 0
- joint base_to_back_right_wheel: axis (none) -> 0 1 0; origin xyz=0 -0.12065 0.0508 -> xyz=0 -0.11 0.05; type fixed -> continuous
- joint base_to_front_left_hinge: axis (none) -> 0 0 1; limit (none) -> lower=-0.5 upper=0.5 effort=10 velocity=100; origin xyz=0.3302 0.12065 0.0508 -> xyz=0.25 0.11 0.05; type fixed -> revolute
- joint base_to_front_right_hinge: axis (none) -> 0 0 1; limit (none) -> lower=-0.5 upper=0.5 effort=10 velocity=100; origin xyz=0.3302 -0.12065 0.0508 -> xyz=0.25 -0.11 0.05; type fixed -> revolute
- joint base_to_laser_model: origin xyz=0.275 0 0.165 -> xyz=0.235 0 0.265
- joint front_left_hinge_to_wheel: axis (none) -> 0 1 0
- joint front_right_hinge_to_wheel: axis (none) -> 0 1 0

File: src/base/robot urdf models/f1tent.xacro (robot description, xacro)
@@ -1,26 +1,22 @@
 <?xml version="1.0"?>
-<!-- A simple model of the racecar for rviz -->
-<robot xmlns:xacro="http://www.ros.org/wiki/xacro" name="racecar">
-  <xacro:property name="wheelbase" value="0.3302" />
-  <xacro:property name="width" value="0.2032" />
-  <xacro:property name="height" value="0.1" />
+<robot xmlns:xacro="http://www.ros.org/wiki/xacro" name="arcpro">
+  <xacro:property name="track_width" value="0.24" />
+  <xacro:property name="body_width" value="0.18" />
+  <xacro:property name="wheelbase" value="0.25" />
+  <xacro:property name="height" value="0.2" />
   <xacro:property name="ground_offset" value="0.04" />
-  <xacro:property name="wheel_radius" value="0.0508" />
-  <xacro:property name="wheel_length" value="0.0381" />
-  <xacro:property name="laser_distance_from_base_link" value="0.275" />
+  <xacro:property name="wheel_radius" value="0.05" />
+  <xacro:property name="wheel_length" value="0.02" />
+  <xacro:property name="laser_distance_from_base_link" value="0.235" />
   <xacro:property name="laser_height" value="0.05" />
   <xacro:property name="laser_radius" value="0.026" />
   <xacro:property name="car_name" value="ego_racecar" />
-  <material name="black">
-    <color rgba="0.2 0.2 0.2 1."/>
-  </material>
-  <material name="blue">
-    <color rgba="0.3 0.57 1. 1."/>
-  </material>
+  <material name="black"><color rgba="0.2 0.2 0.2 1."/></material>
+  <material name="blue"><color rgba="0.3 0.57 1. 1."/></material>
   <link name="${car_name}/base_link">
     <visual>
       <origin xyz="${wheelbase/2} 0 ${ground_offset+height/2}"/>
       <geometry>
-        <box size="${wheelbase} ${width} ${height}"/>
+        <box size="${wheelbase} ${body_width} ${height}"/>
       </geometry>
       <material name="blue"/>
@@ -34,42 +30,61 @@
   <link name="${car_name}/laser_model">
     <visual>
-      <geometry>
-        <cylinder radius="${laser_radius}" length="${laser_height}"/>
-      </geometry>
+      <geometry><cylinder radius="${laser_radius}" length="${laser_height}"/></geometry>
       <material name="black"/>
     </visual>
   </link>
-  <joint name="$base_to_back_left_wheel" type="fixed">
+  <xacro:macro name="wheel" params="name x y rpy type axis">
+    <joint name="${name}_joint" type="${type}">
+      <parent link="${car_name}/base_link"/>
+      <child link="${car_name}/${name}"/>
+      <origin xyz="${x} ${y} ${wheel_radius}"/>
+      <xacro:if value="${type == 'continuous'}">
+        <axis xyz="${axis}"/>
+      </xacro:if>
+      <xacro:if value="${type == 'revolute'}">
+        <axis xyz="${axis}"/>
+        <limit lower="-0.5" upper="0.5" effort="10" velocity="100"/>
+      </xacro:if>
+    </joint>
+    <link name="${car_name}/${name}">
+      <visual>
+        <geometry><cylinder radius="${wheel_radius}" length="${wheel_length}"/></geometry>
+        <material name="black"/>
+        <origin rpy="${rpy}"/>
+      </visual>
+    </link>
+  </xacro:macro>
+  <joint name="base_to_back_left_wheel" type="continuous">
     <parent link="${car_name}/base_link"/>
     <child link="${car_name}/back_left_wheel"/>
-    <origin xyz="0 ${(wheel_length+width)/2} ${wheel_radius}"/>
+    <origin xyz="0 ${track_width/2} ${wheel_radius}"/>
+    <axis xyz="0 1 0"/>
   </joint>
   <link name="${car_name}/back_left_wheel">
     <visual>
-      <geometry>
-        <cylinder radius="${wheel_radius}" length="${wheel_length}"/>
-      </geometry>
+      <geometry><cylinder radius="${wheel_radius}" length="${wheel_length}"/></geometry>
       <material name="black"/>
       <origin rpy="${pi/2} 0 0"/>
     </visual>
   </link>
-  <joint name="base_to_back_right_wheel" type="fixed">
+  <joint name="base_to_back_right_wheel" type="continuous">
     <parent link="${car_name}/base_link"/>
     <child link="${car_name}/back_right_wheel"/>
-    <origin xyz="0 ${-(wheel_length+width)/2} ${wheel_radius}"/>
+    <origin xyz="0 ${-track_width/2} ${wheel_radius}"/>
+    <axis xyz="0 1 0"/>
   </joint>
   <link name="${car_name}/back_right_wheel">
     <visual>
-      <geometry>
-        <cylinder radius="${wheel_radius}" length="${wheel_length}"/>
-      </geometry>
+      <geometry><cylinder radius="${wheel_radius}" length="${wheel_length}"/></geometry>
       <material name="black"/>
       <origin rpy="${pi/2} 0 0"/>
     </visual>
   </link>
-  <joint name="base_to_front_left_hinge" type="fixed">
+  <joint name="base_to_front_left_hinge" type="revolute">
     <parent link="${car_name}/base_link"/>
     <child link="${car_name}/front_left_hinge"/>
-    <origin xyz="${wheelbase} ${(wheel_length+width)/2} ${wheel_radius}"/>
+    <origin xyz="${wheelbase} ${track_width/2} ${wheel_radius}"/>
+    <axis xyz="0 0 1"/>
+    <limit lower="-0.5" upper="0.5" effort="10" velocity="100"/>
   </joint>
   <link name="${car_name}/front_left_hinge"/>
@@ -77,18 +92,19 @@
     <parent link="${car_name}/front_left_hinge"/>
     <child link="${car_name}/front_left_wheel"/>
+    <axis xyz="0 1 0"/>
   </joint>
   <link name="${car_name}/front_left_wheel">
     <visual>
-      <geometry>
-        <cylinder radius="${wheel_radius}" length="${wheel_length}"/>
-      </geometry>
+      <geometry><cylinder radius="${wheel_radius}" length="${wheel_length}"/></geometry>
       <material name="black"/>
       <origin rpy="${pi/2} 0 0"/>
     </visual>
   </link>
-  <joint name="base_to_front_right_hinge" type="fixed">
+  <joint name="base_to_front_right_hinge" type="revolute">
     <parent link="${car_name}/base_link"/>
     <child link="${car_name}/front_right_hinge"/>
-    <origin xyz="${wheelbase} ${-(wheel_length+width)/2} ${wheel_radius}"/>
+    <origin xyz="${wheelbase} ${-track_width/2} ${wheel_radius}"/>
+    <axis xyz="0 0 1"/>
+    <limit lower="-0.5" upper="0.5" effort="10" velocity="100"/>
   </joint>
   <link name="${car_name}/front_right_hinge"/>
@@ -96,10 +112,9 @@
     <parent link="${car_name}/front_right_hinge"/>
     <child link="${car_name}/front_right_wheel"/>
+    <axis xyz="0 1 0"/>
   </joint>
   <link name="${car_name}/front_right_wheel">
     <visual>
-      <geometry>
-        <cylinder radius="${wheel_radius}" length="${wheel_length}"/>
-      </geometry>
+      <geometry><cylinder radius="${wheel_radius}" length="${wheel_length}"/></geometry>
       <material name="black"/>
       <origin rpy="${pi/2} 0 0"/>
